File: eagle/3PCurrentTX.sch (EAGLE design)
At the start: 36 parts, among them IC1 78L05SMD, U1 SN65HVD3082ED, X1 1761543

Commit message: Second commit of Smart EVSE
Parts:
- removed C2: 100n, resistor:C-EUC0805
- removed JP1: (no value), jumper:JP1Q
- removed LED1: 3mm, led:LED3MM
- removed R1: 120R, rcl:R-EU_R0805
- added LED: (no value), led:LEDSML0805
- C1, C10, C4, C5, C6, C7, C8, C9: device resistor:C-EUC0805 -> resistor:C-EUC0805K
- C3: value 47u 16v -> 10u 16v; device resistor:CPOL-EUE2-5 -> resistor:C-EUC1206K
- D1: value 1N4148 -> LL4148
- IC1: value 78L05SMD -> LP2985IM5-5.0; device linear:78L05SMD -> v-reg-micrel:MIC5219XX
- U$1: MPN (none) -> PIC18F14k22-I/SO
- renumbered X1 to RS-485
Connections:
- removed net N$1: JP1.2, R1.1
- net GND: now also C3.2, IC1.GND, LED.C; no longer C2.2, C3.-, IC1G$1.GND@1, IC1G$1.GND@2, IC1G$1.GND@3, IC1G$1.GND@4, LED1.C
- net N$12: no longer R1.2
- net N$13: no longer JP1.1
- net N$15: now also C3.1, IC1.EN, IC1.IN; no longer C2.1, C3.+, IC1G$1.VIN
- net N$8: now also LED.A; no longer LED1.A
- net VCC: now also IC1.OUT; no longer IC1G$1.VOUT
Other:
- note added: "Smart EVSE Sensorbox"
- moved on the sheet: D1
