File: eagle/SmartEVSE.brd (EAGLE design)
At the start: 86.1 x 49.9 mm, 44 parts, among them IC1 78L05SMD, IC2 LM7332MA, IC3 MCP9701A, K2 AQH1213AJ, Q1 16Mhz, U1 PIC18F25K22-I/SO, U2 SN65HVD3082ED, X1 MKDSN1,5/9-5,08, X2 AST027-06

Commit message: Second commit of Smart EVSE
Parts:
- removed JP1: (no value), jumper:JP1
- removed LED: (no value), pinhead:1X02
- removed U1: PIC18F25K22-I/SO, pic_18f25k22:SOIC127P1030X265-28N
- removed U2: SN65HVD3082ED, max487:SOIC127P600X175-8N
- added C13: 100n, rcl:C0805
- added C14: 10000u 16V, rcl:EB22,5D
- added D1, D4: BAT54S, diode:SOT23
- added IC4: PIC18F25K22-I/SOSSOP, pic_18f25k22:SOP65P780X200-28N
- added IC5: SN65HVD3082ED, max487:SOIC127P600X175-8N
- added IC6: TC4424A, tc4424:SOIC127P600X175-8N
- added R14: 100R, resistor:R0805
- added R15: 10K, resistor:R0805
- added R16: 5K1, resistor:R0805
- added U$1: (no value), ohw-logo:OSHW_10X200_NOTEXT
- C1, C2: value 22p -> 18p
- C3: value 100n -> 10u 16v; device rcl:C0805 -> rcl:C1206
- C7: value 10u -> 10u 16v; device rcl:E5-5 -> rcl:C1206
- C9: value 100u -> n.c.; device rcl:E5-5 -> rcl:SMC_C
- IC1: value 78L05SMD -> LP2985IM5-5.0; device linear:SO08 -> v-reg-micrel:SOT23-5
- K1: value AQH1213AJ -> AQH1213AX
- Q1: value 16Mhz -> CTS_32X25_SMD; device special:QS -> cts_crystal:CTS_32X25
- R1: value 120R -> 10K
- R10: value 168R -> 169R
- R12: value 1K -> 1K 1%
- R13: value 330R -> 10K
- R3, R4: value 27K -> 15K
- moved C10 20.0 mm to (68.6, 7.70), turned to 270 degrees
- moved F2 9.10 mm to (76.4, 21.5), turned to 270 degrees
- moved R4 7.77 mm to (57.4, 41.9), turned to 0 degrees
- moved R1 5.44 mm to (69.7, 17.8)
- moved R13 4.91 mm to (73.6, 35.5), turned to 180 degrees
- moved R5 4.80 mm to (60.5, 32.3)
- moved D2 4.70 mm to (73.4, 37.6)
- moved R2 4.50 mm to (52.6, 41.1)
- moved C2 4.47 mm to (69.7, 23.6), turned to 180 degrees
- moved R6 4.40 mm to (70.5, 43.6), turned to 90 degrees
- moved C5 2.90 mm to (51.6, 22.0), turned to 180 degrees
- moved C1 2.67 mm to (69.7, 20.2), turned to 180 degrees
- moved C9 2.55 mm to (44.5, 44.7), flipped to the bottom
- moved R3 2.52 mm to (61.5, 37.1), turned to 90 degrees
- moved Q1 2.43 mm to (66.2, 22.6), flipped to the bottom, turned to 270 degrees
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- renumbered K2 to K1
Connections:
- removed net N$2: JP1.2, R1.1
- removed net N$30: F2.P$2, X1.6
- removed net N$4: R1.2, U2.6, X1.4
- new net N$17: C13.1, C14.+, D1.2, D4.2, IC6.6, R14.2
- new net N$18: IC4.7, IC6.2, R15.1
- new net N$32: F2.P$2, X1.3
- new net N$33: R1.2, X1.5
- new net RS485_A: IC5.6, X1.1
- new net RS485_B: IC5.7, X1.2
- net +12V: now also C7.1, IC1.1, IC1.3, R14.1; no longer C7.+, IC1.8
- net GND: now also C13.2, C14.-, C7.2, D1.1, D4.1, IC4.19, IC4.8, IC5.5, IC6.3, Q1.2, Q1.4, R13.2, R15.2, R16.1, X1.4; no longer C7.-, IC1.3, IC1.6, IC1.7, U1.19, U1.8, U2.5, X1.3, X1.7
- net LCD0: now also IC4.21; no longer U1.21
- net LCD1: now also IC4.22; no longer U1.22
- net LCD2: now also IC4.23; no longer U1.23
- net LCD3: now also IC4.24; no longer U1.24
- net LCD4: now also IC4.11; no longer U1.11
- net LCD6: now also IC4.14; no longer U1.14
- net LCD7: now also IC4.15; no longer U1.15
- net LCD8: now also IC4.16; no longer U1.16
- net N$1: now also IC4.12, R1.1, R16.2; no longer JP1.1, U2.7, X1.5
- net N$11: now also IC4.13; no longer U1.13
- net N$13: now also IC4.2; no longer U1.2
- net N$16: now also IC4.3; no longer U1.3
- net N$20: now also IC4.25; no longer U1.25
- net N$25: now also IC4.26, IC5.2, IC5.3; no longer U1.26, U2.2, U2.3
- net N$27: now also D1.3, IC6.7, X1.6; no longer LED.2, U1.7, X1.1
- net N$28: now also IC4.1; no longer U1.1
- net N$29: now also D4.3, IC6.5, X1.7; no longer LED.1, R13.1, X1.2
- net N$3: now also IC4.6, IC6.4, R13.1; no longer R13.2, U1.6
- net N$31: now also IC4.4; no longer U1.4
- net N$34: now also IC4.28; no longer U1.28
- net N$35: now also IC4.27; no longer U1.27
- net N$5: now also IC4.17, IC5.4; no longer U1.17, U2.4
- net N$6: now also IC4.18, IC5.1; no longer U1.18, U2.1
- net N$7: now also IC4.9, Q1.1; no longer Q1.2, U1.9
- net N$8: now also IC4.10, Q1.3; no longer Q1.1, U1.10
- net VCC: now also IC1.5, IC4.20, IC5.8; no longer IC1.1, U1.20, U2.8
Routing:
- net N$27: track 45.3 -> 7.39 mm
- net N$29: track 33.9 -> 7.51 mm
- net N$17: track 0.00 -> 25.3 mm, vias 0 -> 2
- net N$1: track 31.8 -> 8.79 mm
- net GND: track 79.2 -> 98.8 mm
- net N$4: track 15.1 -> 0.00 mm
- net N$33: track 0.00 -> 13.7 mm
- net N$18: track 0.00 -> 11.8 mm
- net RS485_B: track 0.00 -> 11.1 mm
- net RS485_A: track 0.00 -> 10.3 mm
- net N$25: track 41.0 -> 31.0 mm
- net N$3: track 8.40 -> 18.2 mm
- net N$13: track 18.3 -> 26.1 mm
- net N$34: track 71.1 -> 64.5 mm
- net N$32: track 0.00 -> 6.50 mm
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Other:
- board size 86.1 x 49.9 mm -> 86 x 50 mm
- board text added: "+12V"
- board text added: "A"
- board text added: "B"
- board text added: "CP"
- board text added: "Contactor"
- board text added: "GND"
- board text added: "L1"
- board text added: "N"
- board text added: "PE/GND"
- board text added: "PP"
- board text added: "SOLENOID"
- board text added: "Smart EVSE rev1.3b"
- board text added: "lock"
- board text removed: "Smart EVSE rev1.2"

Commit message: version 1.05, LCD menu added
Parts:
- IC6: value TC4424A -> FAN3214TMX
- R13, R15: value 10K -> NP
Other:
- board text added: "<"
Changed lines of the file:
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@@
 <?xml version="1.0" encoding="utf-8"?>
 <!DOCTYPE eagle SYSTEM "eagle.dtd">
-<eagle version="6.2">
+<eagle version="6.6.0">
 <drawing>
 <settings>
@@
 <wire x1="29.21" y1="16.51" x2="25.4" y2="12.7" width="3.81" layer="26"/>
 <wire x1="25.4" y1="12.7" x2="25.4" y2="2.54" width="3.81" layer="26"/>
+<text x="48.895" y="17.018" size="1.27" layer="25">&lt;</text>
+<text x="52.705" y="8.382" size="1.27" layer="25" rot="R270">&lt;</text>
+<text x="52.578" y="14.732" size="1.27" layer="25" rot="R270">&lt;</text>
 </plain>
 <attributes>
@@
 </class>
 </classes>
-<designrules>
+<designrules name="default">
 <description language="de">&lt;b&gt;EAGLE Design Rules&lt;/b&gt;
 &lt;p&gt;
@@
 <attribute name="VALUE" x="79.015" y="29.633" size="1.27" layer="28" rot="MR0"/>
 </element>
-<element name="IC6" library="tc4424" package="SOIC127P600X175-8N" value="TC4424A" x="71.808" y="31.104" smashed="yes" rot="MR180">
+<element name="IC6" library="tc4424" package="SOIC127P600X175-8N" value="FAN3214TMX" x="71.808" y="31.104" smashed="yes" rot="MR180">
 <attribute name="PACKAGE" value="SOIC-8" x="71.808" y="31.104" size="1.778" layer="28" rot="MR180" display="off"/>
 <attribute name="OC_NEWARK" value="56K7421" x="71.808" y="31.104" size="1.778" layer="28" rot="MR180" display="off"/>
@@
 <attribute name="VALUE" x="73.779" y="24.719" size="1.27" layer="28" rot="MR0"/>
 </element>
-<element name="R13" library="resistor" package="R0805" value="10K" x="73.559" y="35.516" smashed="yes" rot="MR180">
+<element name="R13" library="resistor" package="R0805" value="NP" x="73.559" y="35.516" smashed="yes" rot="MR180">
 <attribute name="NAME" x="75.337" y="36.151" size="1.27" layer="26" rot="MR180"/>
 <attribute name="VALUE" x="72.797" y="37.802" size="1.27" layer="28" rot="MR180"/>
 </element>
-<element name="R15" library="resistor" package="R0805" value="10K" x="68.288" y="27.224" smashed="yes" rot="MR180">
+<element name="R15" library="resistor" package="R0805" value="NP" x="68.288" y="27.224" smashed="yes" rot="MR180">
 <attribute name="NAME" x="65.748" y="26.081" size="1.27" layer="26" rot="MR180"/>
 <attribute name="VALUE" x="67.526" y="29.51" size="1.27" layer="28" rot="MR180"/>
